File: Breakout.kicad_pcb (KiCad board)
At the start: 2 copper layers, 22 x 22 mm, 37 parts, among them K1 easyC-SMD, K2 easyC-SMD, K3 HEADER_MALE_4X1, U1 SE5218, U2 NMOS-DUAL, U3 BME688

Commit message: Add files via upload
Routing:
- net SCL3.3: track 15.9 -> 17.6 mm
- net SCL_PULL5: track 16.5 -> 17.1 mm
- net GND: vias 7 -> 8
Changed lines of the file:
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@@
     (attr board_only exclude_from_pos_files exclude_from_bom)
     (fp_text reference "kibuzzard-640F759F" (at 0 3.678555) (layer "B.SilkS") hide
-      (effects (font (size 0 0)) (justify mirror))
+      (effects (font (size 0 0) (thickness 0.15)) (justify mirror))
     )
     (fp_text value "G***" (at 0 -3.678555) (layer "B.SilkS") hide
-      (effects (font (size 0 0)) (justify mirror))
+      (effects (font (size 0 0) (thickness 0.15)) (justify mirror))
     )
     (fp_poly (pts
@@
   (segment (start 162.45 79.8) (end 161.877 80.373) (width 0.254) (layer "F.Cu") (net 3))
   (segment (start 161.348 80.373) (end 161.025 80.696) (width 0.254) (layer "F.Cu") (net 3))
-  (segment (start 173.015052 68.752) (end 171.785998 68.752) (width 0.254) (layer "F.Cu") (net 4))
-  (segment (start 173.125 68.861948) (end 173.015052 68.752) (width 0.254) (layer "F.Cu") (net 4))
-  (segment (start 173.545148 78.345148) (end 173.575 78.375) (width 0.254) (layer "F.Cu") (net 4))
-  (segment (start 171.785998 68.752) (end 171.3 68.266002) (width 0.254) (layer "F.Cu") (net 4))
+  (segment (start 171.958998 68.925) (end 171.3 68.266002) (width 0.254) (layer "F.Cu") (net 4))
+  (segment (start 174.95 71.025) (end 172.85 68.925) (width 0.254) (layer "F.Cu") (net 4))
+  (segment (start 172.570148 78.9) (end 173.095148 78.375) (width 0.254) (layer "F.Cu") (net 4))
+  (segment (start 172.85 68.925) (end 171.958998 68.925) (width 0.254) (layer "F.Cu") (net 4))
+  (segment (start 173.095148 78.375) (end 173.575 78.375) (width 0.254) (layer "F.Cu") (net 4))
   (segment (start 171.3 68.266002) (end 171.3 66.5) (width 0.254) (layer "F.Cu") (net 4))
-  (segment (start 172.570148 78.345148) (end 173.545148 78.345148) (width 0.254) (layer "F.Cu") (net 4))
-  (segment (start 174.95 71.025) (end 173.125 69.2) (width 0.254) (layer "F.Cu") (net 4))
-  (segment (start 173.125 69.2) (end 173.125 68.861948) (width 0.254) (layer "F.Cu") (net 4))
   (via (at 174.95 71.025) (size 0.5) (drill 0.3) (layers "F.Cu" "B.Cu") (net 4))
-  (via (at 172.570148 78.345148) (size 0.5) (drill 0.3) (layers "F.Cu" "B.Cu") (net 4))
+  (via (at 172.570148 78.9) (size 0.5) (drill 0.3) (layers "F.Cu" "B.Cu") (net 4))
+  (segment (start 174.95 71.2) (end 174.95 71.025) (width 0.254) (layer "B.Cu") (net 4))
+  (segment (start 172.523 78.852852) (end 172.523 72.902) (width 0.254) (layer "B.Cu") (net 4))
   (segment (start 174.35 71.8) (end 174.95 71.2) (width 0.254) (layer "B.Cu") (net 4))
-  (segment (start 172.523 72.902) (end 172.523 78.298) (width 0.254) (layer "B.Cu") (net 4))
+  (segment (start 172.523 72.902) (end 173.625 71.8) (width 0.254) (layer "B.Cu") (net 4))
+  (segment (start 172.570148 78.9) (end 172.523 78.852852) (width 0.254) (layer "B.Cu") (net 4))
   (segment (start 173.625 71.8) (end 174.35 71.8) (width 0.254) (layer "B.Cu") (net 4))
-  (segment (start 172.523 78.298) (end 172.570148 78.345148) (width 0.254) (layer "B.Cu") (net 4))
-  (segment (start 174.95 71.2) (end 174.95 71.025) (width 0.254) (layer "B.Cu") (net 4))
-  (segment (start 172.523 72.902) (end 173.625 71.8) (width 0.254) (layer "B.Cu") (net 4))
   (segment (start 175.925 70.8) (end 172.7 67.575) (width 0.254) (layer "F.Cu") (net 5))
   (segment (start 177.85 72.175) (end 178.5 72.825) (width 0.254) (layer "F.Cu") (net 5))
@@
   (segment (start 173.5 65.425) (end 173.275 65.2) (width 0.254) (layer "F.Cu") (net 7))
   (segment (start 168.75 65.45) (end 168.75 66.5) (width 0.254) (layer "F.Cu") (net 7))
-  (segment (start 169.05 77.575) (end 169.35 77.875) (width 0.254) (layer "F.Cu") (net 8))
-  (segment (start 172.15 77.95) (end 172.875 77.225) (width 0.254) (layer "F.Cu") (net 8))
   (segment (start 169.05 77.55) (end 169.05 76.95) (width 0.254) (layer "F.Cu") (net 8))
-  (segment (start 169.05 76.95) (end 169.05 77.575) (width 0.254) (layer "F.Cu") (net 8))
-  (segment (start 169.425 77.95) (end 171.775 77.95) (width 0.254) (layer "F.Cu") (net 8))
+  (segment (start 175 73.45) (end 175.8 74.25) (width 0.254) (layer "F.Cu") (net 8))
+  (segment (start 172.748 77.728) (end 172.575 77.901) (width 0.254) (layer "F.Cu") (net 8))
   (segment (start 168 78.6) (end 169.05 77.55) (width 0.254) (layer "F.Cu") (net 8))
-  (segment (start 172.875 77.225) (end 173.1 77) (width 0.254) (layer "F.Cu") (net 8))
+  (segment (start 174.375 73.45) (end 175 73.45) (width 0.254) (layer "F.Cu") (net 8))
   (segment (start 164.7 77.1) (end 166.2 78.6) (width 0.254) (layer "F.Cu") (net 8))
-  (segment (start 174.425 74.25) (end 175.8 74.25) (width 0.254) (layer "F.Cu") (net 8))
+  (segment (start 173.7505 77.5) (end 173.5225 77.728) (width 0.254) (layer "F.Cu") (net 8))
   (segment (start 166.2 78.6) (end 168 78.6) (width 0.254) (layer "F.Cu") (net 8))
-  (segment (start 169.35 77.875) (end 169.425 77.95) (width 0.254) (layer "F.Cu") (net 8))
-  (segment (start 174.15 74.525) (end 174.425 74.25) (width 0.254) (layer "F.Cu") (net 8))
-  (segment (start 171.775 77.95) (end 172.15 77.95) (width 0.254) (layer "F.Cu") (net 8))
-  (via (at 174.15 74.525) (size 0.5) (drill 0.3) (layers "F.Cu" "B.Cu") (net 8))
-  (via (at 173.1 77) (size 0.5) (drill 0.3) (layers "F.Cu" "B.Cu") (net 8))
-  (segment (start 174.15 74.525) (end 173.1 75.575) (width 0.254) (layer "B.Cu") (net 8))
-  (segment (start 173.1 75.575) (end 173.1 77) (width 0.254) (layer "B.Cu") (net 8))
-  (segment (start 173.775 75.25) (end 175.8 75.25) (width 0.254) (layer "F.Cu") (net 9))
-  (segment (start 173.35 74.875) (end 173.75 75.275) (width 0.254) (layer "F.Cu") (net 9))
-  (segment (start 173.35 73.7) (end 173.35 74.875) (width 0.254) (layer "F.Cu") (net 9))
+  (segment (start 170.3 78.2) (end 169.05 76.95) (width 0.254) (layer "F.Cu") (net 8))
+  (segment (start 172.575 77.925) (end 172.3 78.2) (width 0.254) (layer "F.Cu") (net 8))
+  (segment (start 172.575 77.901) (end 172.575 77.925) (width 0.254) (layer "F.Cu") (net 8))
+  (segment (start 173.5225 77.728) (end 172.748 77.728) (width 0.254) (layer "F.Cu") (net 8))
+  (segment (start 172.3 78.2) (end 170.3 78.2) (width 0.254) (layer "F.Cu") (net 8))
+  (via (at 174.375 73.45) (size 0.5) (drill 0.3) (layers "F.Cu" "B.Cu") (net 8))
+  (via (at 173.7505 77.5) (size 0.5) (drill 0.3) (layers "F.Cu" "B.Cu") (net 8))
+  (segment (start 174.1 77.1505) (end 173.7505 77.5) (width 0.254) (layer "B.Cu") (net 8))
+  (segment (start 174.1 73.725) (end 174.1 77.1505) (width 0.254) (layer "B.Cu") (net 8))
+  (segment (start 174.375 73.45) (end 174.1 73.725) (width 0.254) (layer "B.Cu") (net 8))
+  (segment (start 170.4745 77.2285) (end 170.823 77.577) (width 0.254) (layer "F.Cu") (net 9))
+  (segment (start 172.85 76.975) (end 173.125 76.7) (width 0.254) (layer "F.Cu") (net 9))
+  (segment (start 174.475 75.25) (end 175.8 75.25) (width 0.254) (layer "F.Cu") (net 9))
   (segment (start 165.32 76.25) (end 165.977 76.907) (width 0.254) (layer "F.Cu") (net 9))
   (segment (start 167.963052 76.720948) (end 167.963052 76.704) (width 0.254) (layer "F.Cu") (net 9))
   (segment (start 167.963052 76.704) (end 168.517052 76.15) (width 0.254) (layer "F.Cu") (net 9))
   (segment (start 167.777 76.907) (end 167.963052 76.720948) (width 0.254) (layer "F.Cu") (net 9))
-  (segment (start 171.825 73.6) (end 173.25 73.6) (width 0.254) (layer "F.Cu") (net 9))
+  (segment (start 173.35 74.125) (end 174.475 75.25) (width 0.254) (layer "F.Cu") (net 9))
   (segment (start 168.517052 76.15) (end 169.05 76.15) (width 0.254) (layer "F.Cu") (net 9))
-  (segment (start 173.25 73.6) (end 173.35 73.7) (width 0.254) (layer "F.Cu") (net 9))
+  (segment (start 172.248 77.577) (end 172.85 76.975) (width 0.254) (layer "F.Cu") (net 9))
   (segment (start 169.05 76.15) (end 170.1245 76.15) (width 0.254) (layer "F.Cu") (net 9))
-  (segment (start 173.75 75.275) (end 173.775 75.25) (width 0.254) (layer "F.Cu") (net 9))
   (segment (start 164.7 76.25) (end 165.32 76.25) (width 0.254) (layer "F.Cu") (net 9))
   (segment (start 170.1245 76.15) (end 170.4745 76.5) (width 0.254) (layer "F.Cu") (net 9))
+  (segment (start 170.823 77.577) (end 172.248 77.577) (width 0.254) (layer "F.Cu") (net 9))
   (segment (start 165.977 76.907) (end 167.777 76.907) (width 0.254) (layer "F.Cu") (net 9))
-  (via (at 170.4745 76.5) (size 0.5) (drill 0.3) (layers "F.Cu" "B.Cu") (net 9))
-  (via (at 171.825 73.6) (size 0.5) (drill 0.3) (layers "F.Cu" "B.Cu") (net 9))
-  (segment (start 171.825 73.6) (end 171.15 73.6) (width 0.254) (layer "B.Cu") (net 9))
-  (segment (start 171.15 73.6) (end 170.75 74) (width 0.254) (layer "B.Cu") (net 9))
-  (segment (start 170.75 76.2245) (end 170.4745 76.5) (width 0.254) (layer "B.Cu") (net 9))
-  (segment (start 170.75 74) (end 170.75 76.2245) (width 0.254) (layer "B.Cu") (net 9))
+  (segment (start 170.4745 76.5) (end 170.4745 77.2285) (width 0.254) (layer "F.Cu") (net 9))
+  (segment (start 173.125 76.7) (end 173.25 76.7) (width 0.254) (layer "F.Cu") (net 9))
+  (via (at 173.35 74.125) (size 0.8) (drill 0.4) (layers "F.Cu" "B.Cu") (net 9))
+  (via (at 173.25 76.7) (size 0.8) (drill 0.4) (layers "F.Cu" "B.Cu") (net 9))
+  (segment (start 173.25 74.225) (end 173.35 74.125) (width 0.254) (layer "B.Cu") (net 9))
+  (segment (start 173.25 76.7) (end 173.25 74.225) (width 0.254) (layer "B.Cu") (net 9))
+  (via (at 175.575 72.775) (size 0.8) (drill 0.4) (layers "F.Cu" "B.Cu") (free) (net 10))
   (via (at 179.925 75.9) (size 0.5) (drill 0.3) (layers "F.Cu" "B.Cu") (free) (net 10))
   (via (at 160.7 76.2) (size 0.5) (drill 0.3) (layers "F.Cu" "B.Cu") (free) (net 10))

Commit message: Add files via upload
Parts:
- removed the G*** at (172.4, 81.5)
- removed the REF** at (171.3, 78.8)
- added REF**: Logo-Front-SolderedFULL-13mm, Soldered Graphics:Logo-Back-SolderedFULL-13mm, F.Cu at (170.3, 75.6)
- added REF**: Logo-Front-Soldered-2.5mm, Soldered Graphics:Logo-Front-Soldered-2.5mm, F.Cu at (171.3, 78.8)
- C1, C2: value 2.2uF -> 2u2
- C3, C4: value 100nF -> 100n
- moved REF** 12.4 mm to (170.2, 82.3)
- moved kibuzzard-640F759F 12.4 mm to (167.7, 82.3)
- moved G*** 11.7 mm to (179.2, 84.3)
- moved R4 0.45 mm to (169.0, 79.7)
Connections:
- net SCL_PULL3,3 renamed SCL_PULL3.3
- net SDA_PULL3,3 renamed SDA_PULL3.3
- R1 pad 2: SDA3,3 -> SDA3.3
- R4 pad 1: SCL3,3 -> SCL3.3
- U2 pad 1: SDA3,3 -> SDA3.3
- U2 pad 4: SCL3,3 -> SCL3.3
Routing:
- net SCL3.3: track 17.6 -> 26.9 mm, vias 2 -> 4
- net SCL3,3: track 7.29 -> 0.00 mm, vias 2 -> 0
- net SDA3.3: track 16.1 -> 23.3 mm
- net SCL_PULL5: track 17.1 -> 15.1 mm
- net SDA3,3: track 1.00 -> 0.00 mm
- net SCL_PULL3.3: track 16.5 -> 17.3 mm
- net SDA_PULL5: track 23.1 -> 23.8 mm
- net GND: vias 8 -> 9
