File: Breakout.kicad_sch (KiCad schematic)
At the start: 20 parts, among them K1 easyC-SMD, K2 easyC-SMD, K3 HEADER_MALE_4X1, U1 SE5218, U2 NMOS-DUAL, U3 BME688

Commit message: Add files via upload
Parts:
- C1, C2: value 2.2uF -> 2u2
- C3, C4: value 100nF -> 100n
Changed lines of the file:
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@@
       (effects (font (size 1.27 1.27)) (justify left))
     )
-    (property "Value" "100nF" (id 1) (at 98.425 125.73 0)
+    (property "Value" "100n" (id 1) (at 98.425 125.73 0)
       (effects (font (size 1.27 1.27)) (justify left))
     )
@@
       (effects (font (size 1.27 1.27)) (justify left))
     )
-    (property "Value" "2.2uF" (id 1) (at 80.01 77.47 0)
+    (property "Value" "2u2" (id 1) (at 80.01 77.47 0)
       (effects (font (size 1.27 1.27)) (justify left))
     )
@@
       (effects (font (size 1.27 1.27)) (justify left))
     )
-    (property "Value" "2.2uF" (id 1) (at 113.03 76.2 0)
+    (property "Value" "2u2" (id 1) (at 113.03 76.2 0)
       (effects (font (size 1.27 1.27)) (justify left))
     )
@@
       (effects (font (size 1.27 1.27)) (justify left))
     )
-    (property "Value" "100nF" (id 1) (at 110.49 125.73 0)
+    (property "Value" "100n" (id 1) (at 110.49 125.73 0)
       (effects (font (size 1.27 1.27)) (justify left))
     )
@@
     )
     (path "/d16641c7-3a7d-4d00-89f3-330697b24f88"
-      (reference "C1") (unit 1) (value "2.2uF") (footprint "e-radionica.com footprinti:0603C")
+      (reference "C1") (unit 1) (value "2u2") (footprint "e-radionica.com footprinti:0603C")
     )
     (path "/c3286fdb-9a55-4d87-8f4d-50f1690a17bf"
-      (reference "C2") (unit 1) (value "2.2uF") (footprint "e-radionica.com footprinti:0603C")
+      (reference "C2") (unit 1) (value "2u2") (footprint "e-radionica.com footprinti:0603C")
     )
     (path "/2e5cc40c-2380-43c9-9f71-e2ad347aef84"
-      (reference "C3") (unit 1) (value "100nF") (footprint "e-radionica.com footprinti:0603C")
+      (reference "C3") (unit 1) (value "100n") (footprint "e-radionica.com footprinti:0603C")
     )
     (path "/fb0b47de-58d4-411f-91f1-1c4a51b99e0c"
-      (reference "C4") (unit 1) (value "100nF") (footprint "e-radionica.com footprinti:0603C")
+      (reference "C4") (unit 1) (value "100n") (footprint "e-radionica.com footprinti:0603C")
     )
     (path "/1802727f-13c6-4551-acdf-415b361a3569"

Commit message: Add files via upload
Connections:
- net SCL3,3 is gone; now on net SCL3.3: R4.1, U2.4 (S1)
- net SDA3,3 is gone; now on net SDA3.3: R1.2, U2.1 (S2)
- net SCL_PULL3,3 renamed SCL_PULL3.3
- net SDA_PULL3,3 renamed SDA_PULL3.3
Changed lines of the file:
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@@
     )
   )
-  (global_label "SDA_PULL3,3" (shape input) (at 171.45 114.935 180) (fields_autoplaced)
+  (global_label "SDA_PULL3.3" (shape input) (at 171.45 114.935 180) (fields_autoplaced)
     (effects (font (size 1.27 1.27)) (justify right))
     (property "Intersheet References" "${INTERSHEET_REFS}" (id 0) (at 156.8207 114.8556 0)
@@
     )
   )
-  (global_label "SDA3,3" (shape input) (at 188.595 111.125 180) (fields_autoplaced)
+  (global_label "SDA3.3" (shape input) (at 188.595 111.125 180) (fields_autoplaced)
     (effects (font (size 1.27 1.27)) (justify right))
     (property "Intersheet References" "${INTERSHEET_REFS}" (id 0) (at 179.59 111.0456 0)
@@
     )
   )
-  (global_label "SCL_PULL3,3" (shape input) (at 230.505 146.05 0) (fields_autoplaced)
+  (global_label "SCL_PULL3.3" (shape input) (at 230.505 146.05 0) (fields_autoplaced)
     (effects (font (size 1.27 1.27)) (justify left))
     (property "Intersheet References" "${INTERSHEET_REFS}" (id 0) (at 245.0738 145.9706 0)
@@
     )
   )
-  (global_label "SCL3,3" (shape input) (at 211.455 124.46 0) (fields_autoplaced)
+  (global_label "SCL3.3" (shape input) (at 211.455 124.46 0) (fields_autoplaced)
     (effects (font (size 1.27 1.27)) (justify left))
     (property "Intersheet References" "${INTERSHEET_REFS}" (id 0) (at 220.3995 124.3806 0)
@@
     )
   )
-  (global_label "SCL_PULL3,3" (shape input) (at 226.695 120.015 0) (fields_autoplaced)
+  (global_label "SCL_PULL3.3" (shape input) (at 226.695 120.015 0) (fields_autoplaced)
     (effects (font (size 1.27 1.27)) (justify left))
     (property "Intersheet References" "${INTERSHEET_REFS}" (id 0) (at 241.2638 119.9356 0)
@@
     )
   )
-  (global_label "SDA_PULL3,3" (shape input) (at 212.725 146.05 180) (fields_autoplaced)
+  (global_label "SDA_PULL3.3" (shape input) (at 212.725 146.05 180) (fields_autoplaced)
     (effects (font (size 1.27 1.27)) (justify right))
     (property "Intersheet References" "${INTERSHEET_REFS}" (id 0) (at 198.0957 145.9706 0)
